File: flipper-pb/flipper-pb.kicad_sch (KiCad schematic)
At the start: 66 parts, among them J1 SWD, J2 UART, J3 LEDS_PWR, J4 UART_PWR, U1 FlipperZero, U2 FlipperZero, X1 SolderPad, X10 SolderPad, X11 SolderPad, X12 SolderPad, X13 SolderPad, X14 SolderPad, X15 SolderPad, X16 SolderPad, X17 SolderPad, X18 SolderPad, X19 SolderPad, X2 SolderPad, X20 SolderPad, X21 SolderPad, X22 SolderPad, X23 SolderPad, X24 SolderPad, X25 SolderPad, X26 SolderPad, X27 SolderPad, X28 SolderPad, X29 SolderPad, X3 SolderPad, X30 SolderPad, X31 SolderPad, X4 SolderPad, X5 SolderPad, X6 SolderPad, X7 SolderPad, X8 SolderPad, X9 SolderPad

Commit message: Diverse Änderungen
Parts:
- removed D10, D9: LED, LED_SMD:LED_0603_1608Metric_Pad1.05x0.95mm_HandSolder, symbol Device:LED
- added C5: 100nF, Capacitor_SMD:C_0603_1608Metric_Pad1.08x0.95mm_HandSolder, symbol Device:C
- added C6: 10uF, Capacitor_SMD:C_0603_1608Metric_Pad1.08x0.95mm_HandSolder, symbol Device:C_Polarized_Small
- added PMOD1: PMOD-Device-x2-Type-1A-GPIO, pmod-conn_6x2:pmod_pin_array_6x2, symbol pmod:PMOD-Device-x2-Type-1A-GPIO
- added PMOD2: PMOD-Device-x2-Type-4A-Expanded-UART, pmod-conn_6x2:pmod_pin_array_6x2, symbol pmod:PMOD-Device-x2-Type-4A-Expanded-UART
- added U3: IIS2DLPCTR, Package_LGA:LGA-12_2x2mm_P0.5mm, symbol Sensor-Nedo:IIS2DLPCTR
- added U4: ISM330DHCX, Package_LGA:LGA-14_3x2.5mm_P0.5mm_LayoutBorder3x4y, symbol Sensor_Motion:ISM330DHCX
- added X32, X33: SolderPad, lomalkin_kicad_footprints:Flipper-SolderPad, symbol lomalkin_kicad_symbols:SolderPad
- R10: value 1K -> 10K
- R9: value 1K -> 10K; now not fitted
Connections:
- net 3.3V: now also R10.1, C5.1, C6.1, PMOD1.12 (VCC), PMOD1.6 (VCC), PMOD2.12 (VCC), PMOD2.6 (VCC), U3.10 (VDDIO), U3.9 (VDD), U4.5 (VDDIO), U4.8 (VDD); no longer X19.1, X20.1
- net GND: now also R9.2, C5.2, C6.2, PMOD1.11 (GND), PMOD1.5 (GND), PMOD2.11 (GND), PMOD2.5 (GND), U3.6 (GND), U3.8 (GND), U4.6 (GND), U4.7 (GND); no longer X25.1, X26.1, X28.1, X29.1
- net PA4: now also PMOD2.8 (RST), U3.12 (INT1), U4.4 (INT1)
- net PA6: now also PMOD2.1 (CTS), U3.3 (SDO/SA0), U4.1 (SDO/SA0)
- net PA7: now also PMOD2.4 (RTS)
- net PC0: now also U3.1 (SCL/SPC), U4.13 (SCL)
- net PC1: now also U3.4 (SDA/SDI/SDO), U4.14 (SDA)
- net PC3: now also PMOD2.7 (INT)
- net SWO: now also U3.11 (INT2), U4.9 (INT2)
- net UART_RX: now also PMOD2.3 (RXD)
- net UART_TX: now also PMOD2.2 (TXD)
- net at J3.2 (Pin_2), R3.1, R4.1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: no longer R10.1, R9.1
- net at R10.2: now also R9.1, U3.2 (CS), U4.12 (CS)
- new net: PMOD1.3 (IOA2), X25.1
- new net: PMOD1.2 (IOA1), X20.1
- new net: PMOD1.4 (IOA3), X26.1
- new net: PMOD1.8 (IOB1), X29.1
- new net: PMOD1.1 (IOA0), X19.1
- new net: PMOD1.10 (IOB3), X33.1
- new net: PMOD1.7 (IOB0), X28.1
- new net: PMOD1.9 (IOB2), X32.1
- no-connect marks 0 -> 1
Other:
- note added: "PA4 (Pin4) can be used as DE/RE Pin for RS485"
- moved on the sheet: R10
